Commit message: Save

File: motoman_description/urdf/sia5/body.urdf.xacro (robot description, xacro)
@@ -130,3 +130,37 @@
     </joint>
   </xacro:macro>
+    <!-- <xacro:macro name="link_v2" params="name mass
+                                      ixx ixy ixz
+                                      iyy iyz izz">
+    <link name="${name}">
+      <visual>
+        <geometry>
+          <mesh filename="package://moveit_resources/panda_description/meshes/visual/${name}.dae"/>
+        </geometry>
+      </visual>
+      <collision>
+        <geometry>
+          <mesh filename="package://moveit_resources/panda_description/meshes/collision/${name}.stl"/>
+        </geometry>
+      </collision>
+      <inertial>
+        <mass value="${mass}"/>
+        <inertia ixx="${ixx}" ixy="${ixy}" ixz="${ixz}" iyy="${iyy}" iyz="${iyz}" izz="${izz}" />
+      </inertial>
+    </link>
+  </xacro:macro>
+  <xacro:macro name="joint_v2" params="joint_name
+                     parent_name child_name
+                                       ox oy oz roll pitch yaw ax ay az
+                     el ll ul vl
+                     skp skv sll sul">
+    <joint name="${joint_name}" type="revolute">
+      <origin xyz="${ox} ${oy} ${oz}" rpy="${roll} ${pitch} ${yaw}"/>
+      <parent link="${parent_name}"/>
+      <child link="${child_name}"/>
+      <axis xyz="${ax} ${ay} ${az}"/>
+    <dynamics damping="0.7" friction="0.7"/>
+      <limit effort="${el}" lower="${ll}" upper="${ul}" velocity="${vl}"/>
+    </joint>
+  </xacro:macro> -->
 </robot>

File: motoman_gazebo/models/urdf/cylinder.urdf (robot description, URDF)
Before this commit: robot cylinder, 1 links, 0 joints
Links:
- link base_link: mass 0.5 -> 1.0; geometry collision cylinder length=0.1 radius=0.03; visual cylinder length=0.1 radius=0.03
