Commit message: Humman control OK

File: dhand_ros_pkg/dhand_description/urdf/base/base.gazebo.xacro (robot description, xacro)
@@ -3,5 +3,5 @@
  <xacro:macro name="dhand_base_gazebo_v0">
   	<gazebo reference="dhand_base_link">
-      <selfCollide>false</selfCollide>
+      <selfCollide>true</selfCollide>
       <mu1 value="0" />
       <mu2 value="0" />

File: dhand_ros_pkg/dhand_description/urdf/base/base.urdf.xacro (robot description, xacro)
@@ -21,32 +21,42 @@
       </inertial>
     </link>
-	<joint name="dhand_palm_joint" type="revolute">
-    <limit velocity="0" effort="0" lower="0" upper="0" />
-	  <origin xyz="0.255 0 0"/>
-	  <parent link="dhand_base_link"/>
-	  <child link="dhand_palm_link"/>
-	</joint>
-  <link name="dhand_palm_link">
-    <collision>
-      <origin xyz="0 0 0" rpy="0 0 0"/>
-      <geometry>
-        <box size="0.005 0.005 0.005"/>
-      </geometry>
-    </collision>
-    <visual>
-      <origin xyz="0 0 0" rpy="0 0 0"/>
-      <geometry>
-        <box size="0.005 0.005 0.005"/>
-      </geometry>
-    </visual>
-    <inertial>
-      <origin xyz="0 0 0" rpy="0 0 0"/>
-      <mass value="1"/>
-      <inertia
-        ixx="0.0" ixy="0.0" ixz="0.0"
-        iyy="0.0" iyz="0.0"
-        izz="0.0"/>
-    </inertial>
-  </link>
+    <joint name="dhand_palm_joint" type="revolute">
+      <limit velocity="0" effort="0" lower="0" upper="0" />
+      <origin xyz="0.255 0 0"/>
+      <parent link="dhand_base_link"/>
+      <child link="dhand_palm_link"/>
+    </joint>
+    <link name="dhand_palm_link">
+      <collision>
+        <origin xyz="0.006 0 0" rpy="0 0 0"/>
+        <geometry>
+          <box size="0.005 0.005 0.005"/>
+        </geometry>
+      </collision>
+      <visual>
+        <origin xyz="0.006 0 0" rpy="0 0 0"/>
+        <geometry>
+          <box size="0.005 0.005 0.005"/>
+        </geometry>
+      </visual>
+      <inertial>
+        <origin xyz="0 0 0" rpy="0 0 0"/>
+        <mass value="1"/>
+        <inertia
+          ixx="0.0" ixy="0.0" ixz="0.0"
+          iyy="0.0" iyz="0.0"
+          izz="0.0"/>
+      </inertial>
+    </link>
+    <transmission name="dhand_palm_transmission">
+      <type>transmission_interface/SimpleTransmission</type>
+      <joint name="dhand_palm_joint">
+		  <hardwareInterface>hardware_interface/PositionJointInterface</hardwareInterface>
+      </joint>
+      <actuator name="dhand_palm_joint_motor">
+        <hardwareInterface>hardware_interface/PositionJointInterface</hardwareInterface>
+        <mechanicalReduction>1</mechanicalReduction>
+      </actuator>
+    </transmission>
   </xacro:macro>
 </robot>
