Commit message: Add dhand grasp fix

File: dhand_ros_pkg/dhand_description/robots/dhand.urdf.xacro (robot description, xacro)
@@ -7,26 +7,26 @@
   <!-- =============== Inertial Info =============== -->
   <xacro:property name="finger_base_mass">
-	<mass value="0.04234931"/>
+	  <mass value="0.04234931"/>
   </xacro:property>
   <xacro:property name="finger_middle_mass">
-	<mass value="0.02332939"/>
+	  <mass value="0.02332939"/>
   </xacro:property>
   <xacro:property name="finger_top_mass">
-	<mass value="0.01452790"/>
+	  <mass value="0.01452790"/>
   </xacro:property>
   <xacro:property name="finger_base_inertia">
-	<inertia ixx="1e-3" ixy="0.00000000" ixz="-0.00001443"
-			 iyy="1e-3" iyz="0.00000000"
-			 izz="1e-3" />
-  </xacro:property>
-  <xacro:property name="finger_middle_inertia">
-	<inertia ixx="1e-3" ixy="0.00000220" ixz="0.00000000"
-			 iyy="1e-3" iyz="0.00000004"
-			 izz="1e-3" />
-  </xacro:property>
-  <xacro:property name="finger_top_inertia">
-	<inertia ixx="1e-3" ixy="0.00000139" ixz="0.00000000"
-			 iyy="1e-3" iyz="0.00000000"
-			 izz="1e-3" />
+    <inertia ixx="1e-3" ixy="0.00000000" ixz="-0.00001443"
+        iyy="1e-3" iyz="0.00000000"
+        izz="1e-3" />
+    </xacro:property>
+    <xacro:property name="finger_middle_inertia">
+    <inertia ixx="1e-3" ixy="0.00000220" ixz="0.00000000"
+        iyy="1e-3" iyz="0.00000004"
+        izz="1e-3" />
+    </xacro:property>
+    <xacro:property name="finger_top_inertia">
+    <inertia ixx="1e-3" ixy="0.00000139" ixz="0.00000000"
+        iyy="1e-3" iyz="0.00000000"
+        izz="1e-3" />
   </xacro:property>
   <!-- =============== Link & Joint =============== -->
@@ -117,3 +117,27 @@
   <xacro:dhand_finger_trans_v0 prefix="top" side="right"/>
   <xacro:dhand_finger_trans_v0 prefix="top" side="left"/>
+  <!-- ====== Gazebo Elements ====== -->
+  <gazebo>
+    <plugin name="gazebo_grasp_fix" filename="libgazebo_grasp_fix.so">
+          <arm>
+            <arm_name>dhand_grasp</arm_name>
+            <palm_link>link_t</palm_link>
+            <gripper_link>dhand_finger_base_right_link</gripper_link>
+            <gripper_link>dhand_finger_base_left_link</gripper_link>
+            <gripper_link>dhand_finger_middle_middle_link</gripper_link>
+            <gripper_link>dhand_finger_middle_right_link</gripper_link>
+            <gripper_link>dhand_finger_middle_left_link</gripper_link>
+            <gripper_link>dhand_finger_top_middle_link</gripper_link>
+            <gripper_link>dhand_finger_top_right_link</gripper_link>
+            <gripper_link>dhand_finger_top_left_link</gripper_link>
+          </arm>
+        <forces_angle_tolerance>100</forces_angle_tolerance>
+        <update_rate>4</update_rate>
+        <grip_count_threshold>4</grip_count_threshold>
+        <max_grip_count>8</max_grip_count>
+        <release_tolerance>0.005</release_tolerance>
+        <disable_collisions_on_attach>false</disable_collisions_on_attach>
+        <contact_topic>__default_topic__</contact_topic>
+      </plugin>
+  </gazebo>
 </robot>

File: dhand_ros_pkg/dhand_description/robots/dhand_adapted.urdf.xacro (robot description, xacro)
@@ -4,7 +4,7 @@
   <xacro:include filename="$(find dhand_description)/urdf/adapter/adapter.urdf.xacro"/>
   <joint name="dhand_base_joint" type="fixed">
-	<origin xyz="0.028 0 0" rpy="0 0 0"/>
-	<parent link="dhand_adapter_link"/>
-	<child link="dhand_base_link"/>
+    <origin xyz="0.028 0 0" rpy="0 0 0"/>
+    <parent link="dhand_adapter_link"/>
+    <child link="dhand_base_link"/>
   </joint>
   <xacro:dhand_adapter_v0/>

File: dhand_ros_pkg/dhand_description/robots/dhand_gazebo.urdf.xacro (robot description, xacro)
@@ -4,7 +4,7 @@
   <link name="world"/>
   <joint name="dhand_adapter_joint" type="fixed">
-	<origin xyz="0 0 0.003" rpy="0 ${-M_PI/2} 0"/>
-	<parent link="world"/>
-	<child link="dhand_adapter_link"/>
+    <origin xyz="0 0 0.003" rpy="0 ${-M_PI/2} 0"/>
+    <parent link="world"/>
+    <child link="dhand_adapter_link"/>
   </joint>
   <!-- ====== Gazebo Elements ====== -->

File: dhand_ros_pkg/dhand_description/urdf/adapter/adapter.gazebo.xacro (robot description, xacro)
@@ -3,7 +3,8 @@
   <xacro:macro name="dhand_adapter_gazebo_v0">
     <gazebo reference="dhand_adapter_link">
-      <mu1>0.8</mu1>
+      <!-- <mu1>0.8</mu1>
       <mu2>0.8</mu2>
-      <selfCollide>false</selfCollide>
+      <selfCollide>false</selfCollide> -->
+      <preserveFixedJoint>true</preserveFixedJoint>
     </gazebo>
   </xacro:macro>

File: dhand_ros_pkg/dhand_description/urdf/base/base.gazebo.xacro (robot description, xacro)
@@ -2,8 +2,9 @@
 <robot xmlns:xacro="http://ros.org/wiki/xacro">
  <xacro:macro name="dhand_base_gazebo_v0">
-	<gazebo reference="dhand_base_link">
-	  <selfCollide>false</selfCollide>
+  	<gazebo reference="dhand_base_link">
+      <selfCollide>false</selfCollide>
       <mu1 value="0.8" />
       <mu2 value="0.8" />
+      <preserveFixedJoint>true</preserveFixedJoint>
     </gazebo>
   </xacro:macro>

File: dhand_ros_pkg/dhand_description/urdf/finger/finger.transmission.xacro (robot description, xacro)
@@ -5,9 +5,9 @@
       <type>transmission_interface/SimpleTransmission</type>
       <joint name="dhand_finger_${prefix}_${side}_joint">
-		<hardwareInterface>hardware_interface/PositionJointInterface</hardwareInterface>
+		  <hardwareInterface>hardware_interface/PositionJointInterface</hardwareInterface>
       </joint>
       <actuator name="dhand_finger_${prefix}_${side}_motor">
-		<hardwareInterface>hardware_interface/PositionJointInterface</hardwareInterface>
-		<mechanicalReduction>1</mechanicalReduction>
+        <hardwareInterface>hardware_interface/PositionJointInterface</hardwareInterface>
+        <mechanicalReduction>1</mechanicalReduction>
       </actuator>
     </transmission>

File: motoman_description/robots/sia5/sia5_basic.urdf.xacro (robot description, xacro)
@@ -1,4 +1,4 @@
 <?xml version="1.0"?>
-<robot name="sia5" xmlns:xacro="http://ros.org/wiki/xacro">
+  <robot name="sia5" xmlns:xacro="http://ros.org/wiki/xacro">
   <!-- File Include -->
   <xacro:include filename="$(find motoman_description)/urdf/common.xacro" />

File: motoman_description/robots/sia5/sia5_with_dhand.urdf.xacro (robot description, xacro)
@@ -15,7 +15,7 @@
   <!-- Joint -->
   <joint name="dhand_adapter_joint" type="fixed">
-	<origin xyz="0 0 0" rpy="${M_PI} 0 0"/>
-	<parent link="tool0"/>
-	<child link="dhand_adapter_link"/>
+    <origin xyz="0 0 0" rpy="0 0 0"/>
+    <parent link="tool0"/>
+    <child link="dhand_adapter_link"/>
   </joint>
 </robot>

File: motoman_description/urdf/common.xacro (robot description, xacro)
@@ -1,4 +1,4 @@
 <?xml version="1.0"?>
 <robot xmlns:xacro="http://ros.org/wiki/xacro">
-    <xacro:property name="M_PI" value="3.14159274" />
+    <xacro:property name="M_PI" value="3.14159265359" />
 </robot>

File: motoman_description/urdf/sia5/body.urdf.xacro (robot description, xacro)
@@ -1,4 +1,4 @@
 <?xml version="1.0"?>
-<robot xmlns:xacro="http://ros.org/wiki/xacro">
+  <robot xmlns:xacro="http://ros.org/wiki/xacro">
   <xacro:property name="sum_rate" value="${base_rate + s_rate
                                       + l_rate + e_rate

File: motoman_gazebo/models/urdf/cylinder.urdf (robot description, URDF)
Before this commit: robot cylinder, 1 links, 0 joints
Links:
- link base_link: geometry collision cylinder length=0.15 radius=0.025; visual cylinder length=0.15 radius=0.025

Commit message: Add dhand palm link to gazeebo for grasp fix

File: dhand_ros_pkg/dhand_description/robots/dhand.urdf.xacro (robot description, xacro)
@@ -117,4 +117,8 @@
   <xacro:dhand_finger_trans_v0 prefix="top" side="right"/>
   <xacro:dhand_finger_trans_v0 prefix="top" side="left"/>
+    <!-- <gazebo reference="dhand_base_link">
+      <disableFixedJointLumping>true</disableFixedJointLumping>
+      <preserveFixedJoint>true</preserveFixedJoint>
+    </gazebo> -->
   <!-- ====== Gazebo Elements ====== -->
   <gazebo>
@@ -122,5 +126,5 @@
           <arm>
             <arm_name>dhand_grasp</arm_name>
-            <palm_link>link_t</palm_link>
+            <palm_link>dhand_palm_link</palm_link>
             <gripper_link>dhand_finger_base_right_link</gripper_link>
             <gripper_link>dhand_finger_base_left_link</gripper_link>

File: dhand_ros_pkg/dhand_description/urdf/adapter/adapter.gazebo.xacro (robot description, xacro)
@@ -3,8 +3,7 @@
   <xacro:macro name="dhand_adapter_gazebo_v0">
     <gazebo reference="dhand_adapter_link">
-      <!-- <mu1>0.8</mu1>
-      <mu2>0.8</mu2>
-      <selfCollide>false</selfCollide> -->
-      <preserveFixedJoint>true</preserveFixedJoint>
+      <selfCollide>false</selfCollide>
+      <mu1>0</mu1>
+      <mu2>0</mu2>
     </gazebo>
   </xacro:macro>

File: dhand_ros_pkg/dhand_description/urdf/base/base.gazebo.xacro (robot description, xacro)
@@ -4,7 +4,6 @@
   	<gazebo reference="dhand_base_link">
       <selfCollide>false</selfCollide>
-      <mu1 value="0.8" />
-      <mu2 value="0.8" />
-      <preserveFixedJoint>true</preserveFixedJoint>
+      <mu1 value="0" />
+      <mu2 value="0" />
     </gazebo>
   </xacro:macro>

File: dhand_ros_pkg/dhand_description/urdf/base/base.urdf.xacro (robot description, xacro)
@@ -21,10 +21,32 @@
       </inertial>
     </link>
-	<joint name="dhand_palm_joint" type="fixed">
+	<joint name="dhand_palm_joint" type="revolute">
+    <limit velocity="0" effort="0" lower="0" upper="0" />
 	  <origin xyz="0.255 0 0"/>
 	  <parent link="dhand_base_link"/>
 	  <child link="dhand_palm_link"/>
 	</joint>
-	<link name="dhand_palm_link"/>
+  <link name="dhand_palm_link">
+    <collision>
+      <origin xyz="0 0 0" rpy="0 0 0"/>
+      <geometry>
+        <box size="0.005 0.005 0.005"/>
+      </geometry>
+    </collision>
+    <visual>
+      <origin xyz="0 0 0" rpy="0 0 0"/>
+      <geometry>
+        <box size="0.005 0.005 0.005"/>
+      </geometry>
+    </visual>
+    <inertial>
+      <origin xyz="0 0 0" rpy="0 0 0"/>
+      <mass value="1"/>
+      <inertia
+        ixx="0.0" ixy="0.0" ixz="0.0"
+        iyy="0.0" iyz="0.0"
+        izz="0.0"/>
+    </inertial>
+  </link>
   </xacro:macro>
 </robot>

Commit message: Go to target obj

File: dhand_ros_pkg/dhand_description/robots/dhand.urdf.xacro (robot description, xacro)
@@ -138,5 +138,5 @@
         <forces_angle_tolerance>100</forces_angle_tolerance>
         <update_rate>4</update_rate>
-        <grip_count_threshold>4</grip_count_threshold>
+        <grip_count_threshold>2</grip_count_threshold>
         <max_grip_count>8</max_grip_count>
         <release_tolerance>0.005</release_tolerance>

File: dhand_ros_pkg/dhand_description/urdf/base/base.urdf.xacro (robot description, xacro)
@@ -21,4 +21,10 @@
       </inertial>
     </link>
+    <joint name="dhand_palmt_joint" type="fixed">
+      <origin xyz="0.255 0 0"/>
+      <parent link="dhand_base_link"/>
+      <child link="dhand_palmt_link"/>
+    </joint>
+    <link name="dhand_palmt_link"/>
     <joint name="dhand_palm_joint" type="revolute">
       <limit velocity="0" effort="0" lower="0" upper="0" />
@@ -29,5 +35,5 @@
     <link name="dhand_palm_link">
       <collision>
-        <origin xyz="0.006 0 0" rpy="0 0 0"/>
+        <origin xyz="0.005 0 0" rpy="0 0 0"/>
         <geometry>
           <box size="0.005 0.005 0.005"/>
@@ -35,5 +41,5 @@
       </collision>
       <visual>
-        <origin xyz="0.006 0 0" rpy="0 0 0"/>
+        <origin xyz="0.005 0 0" rpy="0 0 0"/>
         <geometry>
           <box size="0.005 0.005 0.005"/>
